File: Hardware/PCB_V02/FilamentSpoolScale.kicad_pcb (KiCad board)
At the start: 2 copper layers, 107.2 x 45 mm, 20 parts, among them J1 0.96 inch OLED, J2 Load Cell, J3 Screw_Terminal_01x02, J4 Conn_01x04, J5 Conn_01x07, J6 Conn_01x07, SW1 SW_Push, SW2 SW_Push, SW3 SW_Push

Commit message: PCB correction
Routing:
- net /BT1: track 87.2 -> 90.4 mm
Changed lines of the file:
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@@
   (segment (start 66.4 49.6) (end 69.3 49.6) (width 0.2) (layer "F.Cu") (net 5))
   (segment (start 71.5 49.6) (end 72.5 50.6) (width 0.2) (layer "F.Cu") (net 5))
+  (segment (start 50 62.95) (end 50 59.82) (width 0.25) (layer "F.Cu") (net 5))
   (segment (start 52.56 55.14) (end 53.06 55.14) (width 0.2) (layer "F.Cu") (net 5))
   (segment (start 69.3 49.6) (end 71.5 49.6) (width 0.2) (layer "F.Cu") (net 5))
   (segment (start 72.5 50.6) (end 72.5 53.54) (width 0.2) (layer "F.Cu") (net 5))
+  (segment (start 50 59.82) (end 50.02 59.8) (width 0.25) (layer "F.Cu") (net 5))
   (segment (start 37.4 55.14) (end 53.06 55.14) (width 0.2) (layer "F.Cu") (net 5))
   (via (at 71.5 49.6) (size 0.508) (drill 0.254) (layers "F.Cu" "B.Cu") (free) (net 5))

Commit message: V02 hw
Parts:
- R2: moved to F.Cu
Routing:
- net /BT1: track 90.4 -> 96.9 mm
Changed lines of the file:
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@@
       (net 4 "GND") (pinfunction "1") (pintype "input"))
+  )
+  (footprint "Resistor_THT:R_Axial_DIN0207_L6.3mm_D2.5mm_P10.16mm_Horizontal" (layer "F.Cu")
+    (at 34.1 42.1 -90)
+    (descr "Resistor, Axial_DIN0207 series, Axial, Horizontal, pin pitch=10.16mm, 0.25W = 1/4W, length*diameter=6.3*2.5mm^2, http://cdn-reichelt.de/documents/datenblatt/B400/1_4W%23YAG.pdf")
+    (tags "Resistor Axial_DIN0207 series Axial Horizontal pin pitch 10.16mm 0.25W = 1/4W length 6.3mm diameter 2.5mm")
+    (property "Sheetfile" "FilamentSpoolScale.kicad_sch")
+    (property "Sheetname" "")
+    (attr through_hole)
+    (fp_text reference "R2" (at 5.08 0 90) (layer "F.SilkS")
+      (effects (font (size 1 1) (thickness 0.15)))
+    )
+    (fp_text value "10k" (at 5.08 2.37 90) (layer "F.Fab")
+      (effects (font (size 1 1) (thickness 0.15)))
+    )
+    (fp_text user "${REFERENCE}" (at 5.08 0 90) (layer "F.Fab")
+      (effects (font (size 1 1) (thickness 0.15)))
+    )
+    (fp_line (start 8.35 -1.37) (end 1.81 -1.37) (layer "F.SilkS") (width 0.12))
+    (fp_line (start 8.35 1.37) (end 8.35 -1.37) (layer "F.SilkS") (width 0.12))
+    (fp_line (start 1.81 1.37) (end 8.35 1.37) (layer "F.SilkS") (width 0.12))
+    (fp_line (start 1.04 0) (end 1.81 0) (layer "F.SilkS") (width 0.12))
+    (fp_line (start 9.12 0) (end 8.35 0) (layer "F.SilkS") (width 0.12))
+    (fp_line (start 1.81 -1.37) (end 1.81 1.37) (layer "F.SilkS") (width 0.12))
+    (fp_line (start -1.05 -1.5) (end -1.05 1.5) (layer "F.CrtYd") (width 0.05))
+    (fp_line (start 11.21 -1.5) (end -1.05 -1.5) (layer "F.CrtYd") (width 0.05))
+    (fp_line (start -1.05 1.5) (end 11.21 1.5) (layer "F.CrtYd") (width 0.05))
+    (fp_line (start 11.21 1.5) (end 11.21 -1.5) (layer "F.CrtYd") (width 0.05))
+    (fp_line (start 1.93 -1.25) (end 1.93 1.25) (layer "F.Fab") (width 0.1))
+    (fp_line (start 0 0) (end 1.93 0) (layer "F.Fab") (width 0.1))
+    (fp_line (start 8.23 1.25) (end 8.23 -1.25) (layer "F.Fab") (width 0.1))
+    (fp_line (start 10.16 0) (end 8.23 0) (layer "F.Fab") (width 0.1))
+    (fp_line (start 1.93 1.25) (end 8.23 1.25) (layer "F.Fab") (width 0.1))
+    (fp_line (start 8.23 -1.25) (end 1.93 -1.25) (layer "F.Fab") (width 0.1))
+    (pad "1" thru_hole circle (at 0 0 270) (size 1.6 1.6) (drill 0.8) (layers *.Cu *.Mask)
+      (net 26 "+5V") (pintype "passive"))
+    (pad "2" thru_hole oval (at 10.16 0 270) (size 1.6 1.6) (drill 0.8) (layers *.Cu *.Mask)
+      (net 30 "/BT2") (pintype "passive"))
+    (model "${KICAD6_3DMODEL_DIR}/Resistor_THT.3dshapes/R_Axial_DIN0207_L6.3mm_D2.5mm_P10.16mm_Horizontal.wrl"
+      (offset (xyz 0 0 0))
+      (scale (xyz 1 1 1))
+      (rotate (xyz 0 0 0))
+    )
   )
   (footprint "Button_Switch_THT:SW_PUSH_6mm_H4.3mm" (layer "F.Cu")
@@
     )
   )
-  (footprint "Resistor_THT:R_Axial_DIN0207_L6.3mm_D2.5mm_P10.16mm_Horizontal" (layer "B.Cu")
-    (at 34.1 42.1 -90)
-    (descr "Resistor, Axial_DIN0207 series, Axial, Horizontal, pin pitch=10.16mm, 0.25W = 1/4W, length*diameter=6.3*2.5mm^2, http://cdn-reichelt.de/documents/datenblatt/B400/1_4W%23YAG.pdf")
-    (tags "Resistor Axial_DIN0207 series Axial Horizontal pin pitch 10.16mm 0.25W = 1/4W length 6.3mm diameter 2.5mm")
-    (property "Sheetfile" "FilamentSpoolScale.kicad_sch")
-    (property "Sheetname" "")
-    (attr through_hole)
-    (fp_text reference "R2" (at 5.08 0 90) (layer "B.SilkS")
-      (effects (font (size 1 1) (thickness 0.15)) (justify mirror))
-    )
-    (fp_text value "10k" (at 5.08 -2.37 90) (layer "B.Fab")
-      (effects (font (size 1 1) (thickness 0.15)) (justify mirror))
-    )
-    (fp_text user "${REFERENCE}" (at 5.08 0 90) (layer "B.Fab")
-      (effects (font (size 1 1) (thickness 0.15)) (justify mirror))
-    )
-    (fp_line (start 8.35 1.37) (end 1.81 1.37) (layer "B.SilkS") (width 0.12))
-    (fp_line (start 8.35 -1.37) (end 8.35 1.37) (layer "B.SilkS") (width 0.12))
-    (fp_line (start 1.81 -1.37) (end 8.35 -1.37) (layer "B.SilkS") (width 0.12))
-    (fp_line (start 1.04 0) (end 1.81 0) (layer "B.SilkS") (width 0.12))
-    (fp_line (start 9.12 0) (end 8.35 0) (layer "B.SilkS") (width 0.12))
-    (fp_line (start 1.81 1.37) (end 1.81 -1.37) (layer "B.SilkS") (width 0.12))
-    (fp_line (start -1.05 1.5) (end -1.05 -1.5) (layer "B.CrtYd") (width 0.05))
-    (fp_line (start 11.21 1.5) (end -1.05 1.5) (layer "B.CrtYd") (width 0.05))
-    (fp_line (start -1.05 -1.5) (end 11.21 -1.5) (layer "B.CrtYd") (width 0.05))
-    (fp_line (start 11.21 -1.5) (end 11.21 1.5) (layer "B.CrtYd") (width 0.05))
-    (fp_line (start 1.93 1.25) (end 1.93 -1.25) (layer "B.Fab") (width 0.1))
-    (fp_line (start 0 0) (end 1.93 0) (layer "B.Fab") (width 0.1))
-    (fp_line (start 8.23 -1.25) (end 8.23 1.25) (layer "B.Fab") (width 0.1))
-    (fp_line (start 10.16 0) (end 8.23 0) (layer "B.Fab") (width 0.1))
-    (fp_line (start 1.93 -1.25) (end 8.23 -1.25) (layer "B.Fab") (width 0.1))
-    (fp_line (start 8.23 1.25) (end 1.93 1.25) (layer "B.Fab") (width 0.1))
-    (pad "1" thru_hole circle (at 0 0 270) (size 1.6 1.6) (drill 0.8) (layers *.Cu *.Mask)
-      (net 26 "+5V") (pintype "passive"))
-    (pad "2" thru_hole oval (at 10.16 0 270) (size 1.6 1.6) (drill 0.8) (layers *.Cu *.Mask)
-      (net 30 "/BT2") (pintype "passive"))
-    (model "${KICAD6_3DMODEL_DIR}/Resistor_THT.3dshapes/R_Axial_DIN0207_L6.3mm_D2.5mm_P10.16mm_Horizontal.wrl"
-      (offset (xyz 0 0 0))
-      (scale (xyz 1 1 1))
-      (rotate (xyz 0 0 0))
-    )
-  )
   (gr_line (start 129.5 47.5) (end 129.5 62.5) (layer "Dwgs.User") (width 0.1))
   (gr_line (start 129.5 47.5) (end 84.5 47.5) (layer "Dwgs.User") (width 0.15))
@@
   (segment (start 77.76 55.14) (end 74.1 55.14) (width 0.2) (layer "F.Cu") (net 5))
   (segment (start 60.86 55.14) (end 66.4 49.6) (width 0.2) (layer "F.Cu") (net 5))
+  (segment (start 43.5 62.95) (end 50 62.95) (width 0.25) (layer "F.Cu") (net 5))
   (segment (start 80.1 52.8) (end 77.76 55.14) (width 0.2) (layer "F.Cu") (net 5))
   (segment (start 66.4 49.6) (end 69.3 49.6) (width 0.2) (layer "F.Cu") (net 5))
